Commit message: add support for iqr_topgear

File: husky_description/urdf/decorations.urdf.xacro (robot description, xacro)
@@ -137,5 +137,5 @@
       </xacro:if>
     </xacro:if>
-    <xacro:if value="$(optenv HUSKY_TOP_PLATE_ENABLED true)">
+    <xacro:if value="$(optenv HUSKY_TOP_PLATE_ENABLED false)">
       <!-- Spawn the top plate -->
       <xacro:if value="$(optenv HUSKY_LARGE_TOP_PLATE false)">

File: husky_description/urdf/husky.urdf.xacro (robot description, xacro)
@@ -99,7 +99,7 @@
   <link name="base_footprint"/>
   <joint name="base_footprint_joint" type="fixed">
-    <origin xyz="0 0 ${wheel_vertical_offset - wheel_radius}" rpy="0 0 0" />
-    <parent link="base_link" />
-    <child link="base_footprint" />
+    <origin xyz="0 0 ${wheel_radius - wheel_vertical_offset}" rpy="0 0 0" />
+    <parent link="base_footprint"/>
+    <child link="base_link"/>
   </joint>
   <!-- Inertial link stores the robot's inertial information -->
